File: macropad-01.sch (KiCad schematic (older format))
At the start: 5 parts

Commit message: working through guide
next step is reset button
Parts:
- added C? (x3): 0.1uF, symbol Device:C_Small
- added C?: 10uF, symbol Device:C_Small
- added C? (x2): 22pF, symbol Device:C_Small
- added Y?: 16MHz, symbol Device:Crystal_GND24_Small
Connections:
- wire segments 17 -> 41
Other:
- moved on the sheet: C?, R?, U?

Commit message: schematic complete
Parts:
- added D1, D2, D3, D4: D_Small, Diode_SMD:D_SOD-123, symbol Device:D_Small
- added F1: 500mA, Fuse:Fuse_1206_3216Metric, symbol Device:Polyfuse_Small
- added MX1, MX2, MX3, MX4: MX-NoLED, MX_Alps_Hybrid:MX-1U-NoLED, symbol MX_Alps_Hybrid:MX-NoLED
- added R3: 10k, Resistor_SMD:R_0805_2012Metric, symbol Device:R_Small
- added SW1: SW_Push, random-keyboard-parts:Reset_Pretty, symbol Switch:SW_Push
- added USB1: Molex-0548190589, random-keyboard-parts:Molex-0548190589, symbol random-keyboard-parts:Molex-0548190589
- C1, C2, C3, C4, C5, C6, C7: renamed from C?; footprint (none) -> Capacitor_SMD:C_0805_2012Metric
- R1, R2, R4: renamed from R?; footprint (none) -> Resistor_SMD:R_0805_2012Metric
- Y1: renamed from Y?; footprint (none) -> Crystal:Crystal_SMD_3225-4Pin_3.2x2.5mm
- gave numbers to parts that had none: 1
Connections:
- net labels added: COL0, COL1, D+, D-, ROW0, ROW1, VCC
- wire segments 41 -> 68
